Commit message: URDF: renamed changed box_inertial
... because it doesn't play well with our other URDFs in
kurt_description

File: urdf/sick_tim3xx.urdf.xacro (robot description, xacro)
@@ -5,5 +5,5 @@
   xmlns:xacro="http://ros.org/wiki/xacro"
   name="sick_tim3xx">
-  <xacro:macro name="box_inertial" params="x y z mass origin">
+  <xacro:macro name="box_inertial_with_origin" params="x y z mass origin">
     <inertial>
       <mass value="${mass}" />
@@ -47,5 +47,5 @@
       </geometry>
     </collision>
-    <xacro:box_inertial x="${sick_tim3xx_length}" y="${sick_tim3xx_width}" z="${sick_tim3xx_height}" mass="${sick_tim3xx_mass}" origin="0 0 -0.026" />
+    <xacro:box_inertial_with_origin x="${sick_tim3xx_length}" y="${sick_tim3xx_width}" z="${sick_tim3xx_height}" mass="${sick_tim3xx_mass}" origin="0 0 -0.026" />
   </link>
   <gazebo reference="laser">

Commit message: changed default laser_frame to "laser", made xacro macro

File: urdf/sick_tim3xx.urdf.xacro (robot description, xacro)
@@ -3,6 +3,11 @@
   xmlns:interface="http://playerstage.sourceforge.net/gazebo/xmlschema/#interface"
   xmlns:sensor="http://playerstage.sourceforge.net/gazebo/xmlschema/#sensor"
-  xmlns:xacro="http://ros.org/wiki/xacro"
-  name="sick_tim3xx">
+  xmlns:xacro="http://ros.org/wiki/xacro">
+  <!-- distance between base plate and laser center (= center of mesh) -->
+  <property name="sick_tim3xx_z_offset" value="0.05609" />
+  <property name="sick_tim3xx_length" value="0.06" />
+  <property name="sick_tim3xx_width" value="0.06" />
+  <property name="sick_tim3xx_height" value="0.08" />
+  <property name="sick_tim3xx_mass" value="0.150" />
   <xacro:macro name="box_inertial_with_origin" params="x y z mass origin">
     <inertial>
@@ -14,62 +19,58 @@
     </inertial>
   </xacro:macro>
-  <!-- distance between base plate and laser center (= center of mesh) -->
-  <property name="sick_tim3xx_z_offset" value="0.05609" />
-  <property name="sick_tim3xx_length" value="0.06" />
-  <property name="sick_tim3xx_width" value="0.06" />
-  <property name="sick_tim3xx_height" value="0.08" />
-  <property name="sick_tim3xx_mass" value="0.150" />
-  <link name="laser_mount_link">
-    <inertial>
-      <mass value="0.001" />
-      <origin xyz="0 0 0" />
-      <inertia ixx="0.000001" ixy="0.0" ixz="0.0"
-        iyy="0.000001" iyz="0.0" izz="0.000001" />
-    </inertial>
-  </link>
-  <joint name="laser_joint" type="fixed">
-    <parent link="laser_mount_link" />
-    <child link="laser_link" />
-    <origin rpy="0 0 0" xyz="0 0 ${sick_tim3xx_z_offset}"/>
-  </joint>
-  <link name="laser_link">
-    <visual>
-      <geometry>
-        <mesh filename="package://sick_tim3xx/meshes/sick_tim3xx.stl" />
-      </geometry>
-      <material name="blue" >
-        <color rgba="0 0 1 1" />
-      </material>
-    </visual>
-    <collision>
-      <geometry>
-        <mesh filename="package://sick_tim3xx/meshes/sick_tim3xx.stl" />
-      </geometry>
-    </collision>
-    <xacro:box_inertial_with_origin x="${sick_tim3xx_length}" y="${sick_tim3xx_width}" z="${sick_tim3xx_height}" mass="${sick_tim3xx_mass}" origin="0 0 -0.026" />
-  </link>
-  <gazebo reference="laser_link">
-    <material value="Gazebo/Blue" />
-    <sensor:ray name="laser">
-      <rayCount>271</rayCount>
-      <rangeCount>271</rangeCount>
-      <laserCount>1</laserCount>
-      <origin>0.0 0.0 0.0</origin>
-      <displayRays>false</displayRays>
-      <minAngle>-135</minAngle>
-      <maxAngle>135</maxAngle>
-      <minRange>0.05</minRange>
-      <maxRange>4.0</maxRange>
-      <resRange>0.01</resRange>
-      <updateRate>15.0</updateRate>
-      <controller:gazebo_ros_laser name="gazebo_ros_laser_controller" plugin="libgazebo_ros_laser.so">
-        <gaussianNoise>0.005</gaussianNoise>
-        <alwaysOn>true</alwaysOn>
+  <xacro:macro name="sick_tim3xx" params="laser_link">
+    <link name="laser_mount_link">
+      <inertial>
+        <mass value="0.001" />
+        <origin xyz="0 0 0" />
+        <inertia ixx="0.000001" ixy="0.0" ixz="0.0"
+          iyy="0.000001" iyz="0.0" izz="0.000001" />
+      </inertial>
+    </link>
+    <joint name="laser_joint" type="fixed">
+      <parent link="laser_mount_link" />
+      <child link="${laser_link}" />
+      <origin rpy="0 0 0" xyz="0 0 ${sick_tim3xx_z_offset}"/>
+    </joint>
+    <link name="${laser_link}">
+      <visual>
+        <geometry>
+          <mesh filename="package://sick_tim3xx/meshes/sick_tim3xx.stl" />
+        </geometry>
+        <material name="blue" >
+          <color rgba="0 0 1 1" />
+        </material>
+      </visual>
+      <collision>
+        <geometry>
+          <mesh filename="package://sick_tim3xx/meshes/sick_tim3xx.stl" />
+        </geometry>
+      </collision>
+      <xacro:box_inertial_with_origin x="${sick_tim3xx_length}" y="${sick_tim3xx_width}" z="${sick_tim3xx_height}" mass="${sick_tim3xx_mass}" origin="0 0 -0.026" />
+    </link>
+    <gazebo reference="${laser_link}">
+      <material value="Gazebo/Blue" />
+      <sensor:ray name="laser">
+        <rayCount>271</rayCount>
+        <rangeCount>271</rangeCount>
+        <laserCount>1</laserCount>
+        <origin>0.0 0.0 0.0</origin>
+        <displayRays>false</displayRays>
+        <minAngle>-135</minAngle>
+        <maxAngle>135</maxAngle>
+        <minRange>0.05</minRange>
+        <maxRange>4.0</maxRange>
+        <resRange>0.01</resRange>
         <updateRate>15.0</updateRate>
-        <topicName>scan</topicName>
-        <frameName>laser_link</frameName>
-        <interface:laser name="gazebo_ros_laser_iface" />
-      </controller:gazebo_ros_laser>
-    </sensor:ray>
-  </gazebo>
+        <controller:gazebo_ros_laser name="gazebo_ros_laser_controller" plugin="libgazebo_ros_laser.so">
+          <gaussianNoise>0.005</gaussianNoise>
+          <alwaysOn>true</alwaysOn>
+          <updateRate>15.0</updateRate>
+          <topicName>scan</topicName>
+          <frameName>${laser_link}</frameName>
+          <interface:laser name="gazebo_ros_laser_iface" />
+        </controller:gazebo_ros_laser>
+      </sensor:ray>
+    </gazebo>
+  </xacro:macro>
 </robot>

Commit message: update URDF to be compatible with Gazebo 1.5
In the ros-groovy-simulator-gazebo update to 1.7.12, Gazebo was switched
over to 1.5, which breaks compatibility with old-style URDFs. This
commit updates to the new version.

File: urdf/sick_tim3xx.urdf.xacro (robot description, xacro)
@@ -49,27 +49,37 @@
       <xacro:box_inertial_with_origin x="${sick_tim3xx_length}" y="${sick_tim3xx_width}" z="${sick_tim3xx_height}" mass="${sick_tim3xx_mass}" origin="0 0 -0.026" />
     </link>
-    <gazebo reference="${laser_link}">
+    <xacro:sick_tim3xx_laser_gazebo_v0 name="laser" link="${laser_link}" ros_topic="scan" update_rate="15.0" min_angle="-2.357" max_angle="2.357" />
+  </xacro:macro>
+  <xacro:macro name="sick_tim3xx_laser_gazebo_v0" params="name link ros_topic update_rate min_angle max_angle">
+    <gazebo reference="${link}">
       <material value="Gazebo/Blue" />
-      <sensor:ray name="laser">
-        <rayCount>271</rayCount>
-        <rangeCount>271</rangeCount>
-        <laserCount>1</laserCount>
-        <origin>0.0 0.0 0.0</origin>
-        <displayRays>false</displayRays>
-        <minAngle>-135</minAngle>
-        <maxAngle>135</maxAngle>
-        <minRange>0.05</minRange>
-        <maxRange>4.0</maxRange>
-        <resRange>0.01</resRange>
-        <updateRate>15.0</updateRate>
-        <controller:gazebo_ros_laser name="gazebo_ros_laser_controller" plugin="libgazebo_ros_laser.so">
+      <sensor type="ray" name="${name}">
+        <always_on>true</always_on>
+        <update_rate>${update_rate}</update_rate>
+        <pose>0 0 0 0 0 0</pose>
+        <visualize>false</visualize>
+        <ray>
+          <scan>
+            <horizontal>
+              <samples>271</samples>
+              <resolution>1</resolution>
+              <min_angle>${min_angle}</min_angle>
+              <max_angle>${max_angle}</max_angle>
+            </horizontal>
+          </scan>
+          <range>
+            <min>0.05</min>
+            <max>4.0</max>
+            <resolution>0.01</resolution>
+          </range>
+        </ray>
+        <plugin name="gazebo_ros_${name}_controller" filename="libgazebo_ros_laser.so">
           <gaussianNoise>0.005</gaussianNoise>
           <alwaysOn>true</alwaysOn>
-          <updateRate>15.0</updateRate>
-          <topicName>scan</topicName>
-          <frameName>${laser_link}</frameName>
-          <interface:laser name="gazebo_ros_laser_iface" />
-        </controller:gazebo_ros_laser>
-      </sensor:ray>
+          <updateRate>${update_rate}</updateRate>
+          <topicName>${ros_topic}</topicName>
+          <frameName>${link}</frameName>
+        </plugin>
+      </sensor>
     </gazebo>
   </xacro:macro>

Commit message: urdf: removed box_inertial_with_origin xacro macro
this conflicted with a new macro of the same name in
uos_common_urdf/common.xacro

File: urdf/sick_tim3xx.urdf.xacro (robot description, xacro)
@@ -10,13 +10,4 @@
   <property name="sick_tim3xx_height" value="0.08" />
   <property name="sick_tim3xx_mass" value="0.150" />
-  <xacro:macro name="box_inertial_with_origin" params="x y z mass origin">
-    <inertial>
-      <mass value="${mass}" />
-      <origin xyz="${origin}" />
-      <inertia ixx="${0.0833333 * mass * (y*y + z*z)}" ixy="0.0" ixz="0.0"
-        iyy="${0.0833333 * mass * (x*x + z*z)}" iyz="0.0"
-        izz="${0.0833333 * mass * (x*x + y*y)}" />
-    </inertial>
-  </xacro:macro>
   <xacro:macro name="sick_tim3xx" params="laser_link">
     <link name="laser_mount_link">
@@ -47,5 +38,11 @@
         </geometry>
       </collision>
-      <xacro:box_inertial_with_origin x="${sick_tim3xx_length}" y="${sick_tim3xx_width}" z="${sick_tim3xx_height}" mass="${sick_tim3xx_mass}" origin="0 0 -0.026" />
+      <inertial>
+        <mass value="${sick_tim3xx_mass}" />
+        <origin xyz="0 0 -0.026" />
+        <inertia ixx="${0.0833333 * sick_tim3xx_mass * (sick_tim3xx_width * sick_tim3xx_width + sick_tim3xx_height * sick_tim3xx_height)}" ixy="0.0" ixz="0.0"
+          iyy="${0.0833333 * sick_tim3xx_mass * (sick_tim3xx_length * sick_tim3xx_length + sick_tim3xx_height * sick_tim3xx_height)}" iyz="0.0"
+          izz="${0.0833333 * sick_tim3xx_mass * (sick_tim3xx_length * sick_tim3xx_length + sick_tim3xx_width * sick_tim3xx_width)}" />
+      </inertial>
     </link>
     <xacro:sick_tim3xx_laser_gazebo_v0 name="laser" link="${laser_link}" ros_topic="scan" update_rate="15.0" min_angle="-2.357" max_angle="2.357" />

Commit message: urdf: removed box_inertial_with_origin xacro macro
this conflicted with a new macro of the same name in
uos_common_urdf/common.xacro

Conflicts:
	urdf/sick_tim3xx.urdf.xacro

File: urdf/sick_tim3xx.urdf.xacro (robot description, xacro)
@@ -10,13 +10,4 @@
   <property name="sick_tim3xx_height" value="0.08" />
   <property name="sick_tim3xx_mass" value="0.150" />
-  <xacro:macro name="box_inertial_with_origin" params="x y z mass origin">
-    <inertial>
-      <mass value="${mass}" />
-      <origin xyz="${origin}" />
-      <inertia ixx="${0.0833333 * mass * (y*y + z*z)}" ixy="0.0" ixz="0.0"
-        iyy="${0.0833333 * mass * (x*x + z*z)}" iyz="0.0"
-        izz="${0.0833333 * mass * (x*x + y*y)}" />
-    </inertial>
-  </xacro:macro>
   <xacro:macro name="sick_tim3xx" params="laser_link">
     <link name="laser_mount_link">
@@ -47,5 +38,11 @@
         </geometry>
       </collision>
-      <xacro:box_inertial_with_origin x="${sick_tim3xx_length}" y="${sick_tim3xx_width}" z="${sick_tim3xx_height}" mass="${sick_tim3xx_mass}" origin="0 0 -0.026" />
+      <inertial>
+        <mass value="${sick_tim3xx_mass}" />
+        <origin xyz="0 0 -0.026" />
+        <inertia ixx="${0.0833333 * sick_tim3xx_mass * (sick_tim3xx_width * sick_tim3xx_width + sick_tim3xx_height * sick_tim3xx_height)}" ixy="0.0" ixz="0.0"
+          iyy="${0.0833333 * sick_tim3xx_mass * (sick_tim3xx_length * sick_tim3xx_length + sick_tim3xx_height * sick_tim3xx_height)}" iyz="0.0"
+          izz="${0.0833333 * sick_tim3xx_mass * (sick_tim3xx_length * sick_tim3xx_length + sick_tim3xx_width * sick_tim3xx_width)}" />
+      </inertial>
     </link>
     <gazebo reference="${laser_link}">

Commit message: added parameters for the name, the laser_link and the ros topic

File: urdf/sick_tim3xx.urdf.xacro (robot description, xacro)
@@ -10,5 +10,5 @@
   <property name="sick_tim3xx_height" value="0.08" />
   <property name="sick_tim3xx_mass" value="0.150" />
-  <xacro:macro name="sick_tim3xx" params="laser_link">
+  <xacro:macro name="sick_tim3xx" params="name ros_topic laser_link">
     <link name="laser_mount_link">
       <inertial>
@@ -46,5 +46,5 @@
       </inertial>
     </link>
-    <xacro:sick_tim3xx_laser_gazebo_v0 name="laser" link="${laser_link}" ros_topic="scan" update_rate="15.0" min_angle="-2.357" max_angle="2.357" />
+    <xacro:sick_tim3xx_laser_gazebo_v0 name="${name}" link="${laser_link}" ros_topic="${ros_topic}" update_rate="15.0" min_angle="-2.357" max_angle="2.357" />
   </xacro:macro>
   <xacro:macro name="sick_tim3xx_laser_gazebo_v0" params="name link ros_topic update_rate min_angle max_angle">
