Commit message: completed rename: sick_tim3xx -> sick_tim
    perl -e 's/sick_tim3xx/sick_tim/g' -pi $(git ls-files)
    perl -e 's/SickTim3xx/SickTim/g' -pi $(git ls-files)
    rename 's/sick_tim3xx/sick_tim/g' $(git ls-files)
    rename 's/SickTim3xx/SickTim/g' $(git ls-files)

File: urdf/sick_tim.urdf.xacro (robot description, xacro)
@@ -5,10 +5,10 @@
   xmlns:xacro="http://ros.org/wiki/xacro">
   <!-- distance between base plate and laser center (= center of mesh) -->
-  <property name="sick_tim3xx_z_offset" value="0.05609" />
-  <property name="sick_tim3xx_length" value="0.06" />
-  <property name="sick_tim3xx_width" value="0.06" />
-  <property name="sick_tim3xx_height" value="0.08" />
-  <property name="sick_tim3xx_mass" value="0.150" />
-  <xacro:macro name="sick_tim3xx" params="laser_link">
+  <property name="sick_tim_z_offset" value="0.05609" />
+  <property name="sick_tim_length" value="0.06" />
+  <property name="sick_tim_width" value="0.06" />
+  <property name="sick_tim_height" value="0.08" />
+  <property name="sick_tim_mass" value="0.150" />
+  <xacro:macro name="sick_tim" params="laser_link">
     <link name="laser_mount_link">
       <inertial>
@@ -22,10 +22,10 @@
       <parent link="laser_mount_link" />
       <child link="${laser_link}" />
-      <origin rpy="0 0 0" xyz="0 0 ${sick_tim3xx_z_offset}"/>
+      <origin rpy="0 0 0" xyz="0 0 ${sick_tim_z_offset}"/>
     </joint>
     <link name="${laser_link}">
       <visual>
         <geometry>
-          <mesh filename="package://sick_tim3xx/meshes/sick_tim3xx.stl" />
+          <mesh filename="package://sick_tim/meshes/sick_tim.stl" />
         </geometry>
         <material name="blue" >
@@ -35,13 +35,13 @@
       <collision>
         <geometry>
-          <mesh filename="package://sick_tim3xx/meshes/sick_tim3xx.stl" />
+          <mesh filename="package://sick_tim/meshes/sick_tim.stl" />
         </geometry>
       </collision>
       <inertial>
-        <mass value="${sick_tim3xx_mass}" />
+        <mass value="${sick_tim_mass}" />
         <origin xyz="0 0 -0.026" />
-        <inertia ixx="${0.0833333 * sick_tim3xx_mass * (sick_tim3xx_width * sick_tim3xx_width + sick_tim3xx_height * sick_tim3xx_height)}" ixy="0.0" ixz="0.0"
-          iyy="${0.0833333 * sick_tim3xx_mass * (sick_tim3xx_length * sick_tim3xx_length + sick_tim3xx_height * sick_tim3xx_height)}" iyz="0.0"
-          izz="${0.0833333 * sick_tim3xx_mass * (sick_tim3xx_length * sick_tim3xx_length + sick_tim3xx_width * sick_tim3xx_width)}" />
+        <inertia ixx="${0.0833333 * sick_tim_mass * (sick_tim_width * sick_tim_width + sick_tim_height * sick_tim_height)}" ixy="0.0" ixz="0.0"
+          iyy="${0.0833333 * sick_tim_mass * (sick_tim_length * sick_tim_length + sick_tim_height * sick_tim_height)}" iyz="0.0"
+          izz="${0.0833333 * sick_tim_mass * (sick_tim_length * sick_tim_length + sick_tim_width * sick_tim_width)}" />
       </inertial>
     </link>

Commit message: updated URDF: restructuring, add TiM 511
Conflicts:
	urdf/sick_tim.urdf.xacro

File: urdf/sick_tim.urdf.xacro (robot description, xacro)
@@ -4,12 +4,19 @@
   xmlns:sensor="http://playerstage.sourceforge.net/gazebo/xmlschema/#sensor"
   xmlns:xacro="http://ros.org/wiki/xacro">
-  <!-- distance between base plate and laser center (= center of mesh) -->
-  <property name="sick_tim_z_offset" value="0.05609" />
-  <property name="sick_tim_length" value="0.06" />
-  <property name="sick_tim_width" value="0.06" />
-  <property name="sick_tim_height" value="0.08" />
-  <property name="sick_tim_mass" value="0.150" />
-  <xacro:macro name="sick_tim" params="laser_link">
-    <link name="laser_mount_link">
+  <xacro:macro name="sick_tim310" params="name ros_topic">
+    <xacro:sick_tim name="${name}" ros_topic="${ros_topic}"
+      length="0.06" width="0.06" height="0.79" mass="0.150" z_offset="0.05595"
+      min_range="0.05" max_range="4.0"
+      mesh="package://sick_tim/meshes/sick_tim310.stl" />
+  </xacro:macro>
+  <xacro:macro name="sick_tim551" params="name ros_topic">
+    <xacro:sick_tim name="${name}" ros_topic="${ros_topic}"
+      length="0.06" width="0.06" height="0.86" mass="0.250" z_offset="0.06296"
+      min_range="0.05" max_range="10.0"
+      mesh="package://sick_tim/meshes/sick_tim551.stl" />
+  </xacro:macro>
+  <xacro:macro name="sick_tim" params="name ros_topic length width height mass z_offset min_range max_range mesh">
+    <!-- z_offset: distance between base plate and laser center (= center of mesh) -->
+    <link name="${name}_mount_link">
       <inertial>
         <mass value="0.001" />
@@ -19,13 +26,13 @@
       </inertial>
     </link>
-    <joint name="laser_joint" type="fixed">
-      <parent link="laser_mount_link" />
-      <child link="${laser_link}" />
-      <origin rpy="0 0 0" xyz="0 0 ${sick_tim_z_offset}"/>
+    <joint name="${name}_joint" type="fixed">
+      <parent link="${name}_mount_link" />
+      <child link="${name}" />
+      <origin rpy="0 0 0" xyz="0 0 ${z_offset}"/>
     </joint>
-    <link name="${laser_link}">
+    <link name="${name}">
       <visual>
         <geometry>
-          <mesh filename="package://sick_tim/meshes/sick_tim.stl" />
+          <mesh filename="${mesh}" />
         </geometry>
         <material name="blue" >
@@ -35,18 +42,18 @@
       <collision>
         <geometry>
-          <mesh filename="package://sick_tim/meshes/sick_tim.stl" />
+          <mesh filename="${mesh}" />
         </geometry>
       </collision>
       <inertial>
-        <mass value="${sick_tim_mass}" />
+        <mass value="${mass}" />
         <origin xyz="0 0 -0.026" />
-        <inertia ixx="${0.0833333 * sick_tim_mass * (sick_tim_width * sick_tim_width + sick_tim_height * sick_tim_height)}" ixy="0.0" ixz="0.0"
-          iyy="${0.0833333 * sick_tim_mass * (sick_tim_length * sick_tim_length + sick_tim_height * sick_tim_height)}" iyz="0.0"
-          izz="${0.0833333 * sick_tim_mass * (sick_tim_length * sick_tim_length + sick_tim_width * sick_tim_width)}" />
+        <inertia ixx="${0.0833333 * mass * (width * width + height * height)}" ixy="0.0" ixz="0.0"
+          iyy="${0.0833333 * mass * (length * length + height * height)}" iyz="0.0"
+          izz="${0.0833333 * mass * (length * length + width * width)}" />
       </inertial>
     </link>
-    <xacro:sick_tim3xx_laser_gazebo_v0 name="laser" link="${laser_link}" ros_topic="scan" update_rate="15.0" min_angle="-2.357" max_angle="2.357" />
+    <xacro:sick_tim_laser_gazebo_v0 name="${name}" link="${name}" ros_topic="${ros_topic}" update_rate="15.0" min_angle="-2.357" max_angle="2.357" min_range="${min_range}" max_range="${max_range}"/>
   </xacro:macro>
-  <xacro:macro name="sick_tim3xx_laser_gazebo_v0" params="name link ros_topic update_rate min_angle max_angle">
+  <xacro:macro name="sick_tim_laser_gazebo_v0" params="name link ros_topic update_rate min_angle max_angle min_range max_range">
     <gazebo reference="${link}">
       <material value="Gazebo/Blue" />
@@ -66,6 +73,6 @@
           </scan>
           <range>
-            <min>0.05</min>
-            <max>4.0</max>
+            <min>${min_range}</min>
+            <max>${max_range}</max>
             <resolution>0.01</resolution>
           </range>

Commit message: Make view angle configurable

File: urdf/sick_tim.urdf.xacro (robot description, xacro)
@@ -10,11 +10,12 @@
       mesh="package://sick_tim/meshes/sick_tim310.stl" />
   </xacro:macro>
-  <xacro:macro name="sick_tim551" params="name ros_topic">
+  <xacro:macro name="sick_tim551" params="name ros_topic min_angle:=-1.5707 max_angle:=1.5707 min_range:=0.05 max_range:=10">
     <xacro:sick_tim name="${name}" ros_topic="${ros_topic}"
       length="0.06" width="0.06" height="0.086" mass="0.250" z_offset="0.06296"
-      min_range="0.05" max_range="10.0"
+      min_range="${min_range}" max_range="${max_range}"
+      min_angle="${min_angle}" max_angle="${max_angle}"
       mesh="package://sick_tim/meshes/sick_tim551.stl" />
   </xacro:macro>
-  <xacro:macro name="sick_tim" params="name ros_topic length width height mass z_offset min_range max_range mesh">
+  <xacro:macro name="sick_tim" params="name ros_topic length width height mass z_offset min_angle max_angle min_range max_range mesh">
     <!-- z_offset: distance between base plate and laser center (= center of mesh) -->
     <link name="${name}_mount_link">
@@ -53,5 +54,5 @@
       </inertial>
     </link>
-    <xacro:sick_tim_laser_gazebo_v0 name="${name}" link="${name}" ros_topic="${ros_topic}" update_rate="15.0" min_angle="-2.357" max_angle="2.357" min_range="${min_range}" max_range="${max_range}"/>
+    <xacro:sick_tim_laser_gazebo_v0 name="${name}" link="${name}" ros_topic="${ros_topic}" update_rate="15.0" min_angle="${min_angle}" max_angle="${max_angle}" min_range="${min_range}" max_range="${max_range}"/>
   </xacro:macro>
   <xacro:macro name="sick_tim_laser_gazebo_v0" params="name link ros_topic update_rate min_angle max_angle min_range max_range">
